Commit message: cambio umbral

File: turtlebot3/tb3_descriptions/turtlebot3_burger_for_autorace.urdf.xacro (robot description, xacro)
@@ -141,5 +141,5 @@
   </link>
   <joint name="camera_joint" type="fixed">
-    <origin xyz="0.00 -0.011 0.130" rpy="0 0.45 0"/>
+    <origin xyz="0.00 -0.011 0.130" rpy="0 0.6 0"/>
     <parent link="base_link"/>
     <child link="camera_link"/>
