Commit message: axustada camara, rexion de reforzo, segundo aproximacion qlearning

File: turtlebot3/tb3_descriptions/turtlebot3_burger_for_autorace.gazebo.xacro (robot description, xacro)
@@ -143,5 +143,5 @@
       <plugin name="camera_controller" filename="libgazebo_ros_camera.so">
         <alwaysOn>true</alwaysOn>
-        <updateRate>30.0</updateRate>
+        <updateRate>10.0</updateRate>
         <cameraName>camera</cameraName>
         <frameName>camera_rgb_optical_frame</frameName>

File: turtlebot3/tb3_descriptions/turtlebot3_burger_for_autorace.urdf.xacro (robot description, xacro)
@@ -141,5 +141,5 @@
   </link>
   <joint name="camera_joint" type="fixed">
-    <origin xyz="0.00 -0.011 0.130" rpy="0 0.6 0"/>
+    <origin xyz="0.008 -0.011 0.130" rpy="0 0.6 0"/>
     <parent link="base_link"/>
     <child link="camera_link"/>
